File: Hardware/TSL238T-breakout.brd (EAGLE design)
At the start: 15 x 15 mm, 4 parts, among them J1 CONN_42.54_NOSILK

Commit message: Labels, 3rd hole
Parts:
- added H3: (no value), bschulz:2_56
Connections:
- net N$1 renamed GND
- net N$2 renamed VDD
- net N$3 renamed OE
- net N$4 renamed OUT
Other:
- board text added: "GND"
- board text added: "OE"
- board text added: "OUT"
- board text added: "VDD"
Changed lines of the file:
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@@
 <?xml version="1.0" encoding="utf-8"?>
 <!DOCTYPE eagle SYSTEM "eagle.dtd">
-<eagle version="9.2.2">
+<eagle version="9.2.0">
 <drawing>
 <settings>
@@
 <wire x1="0" y1="13" x2="0" y2="2" width="0" layer="20"/>
 <wire x1="0" y1="2" x2="2" y2="0" width="0" layer="20" curve="90"/>
+<text x="1.8" y="2.5" size="0.8128" layer="52" rot="MR90">VDD</text>
+<text x="9.3" y="2.5" size="0.8128" layer="52" rot="MR90">OUT</text>
+<text x="4.3" y="2.5" size="0.8128" layer="52" rot="MR90">GND</text>
+<text x="6.8" y="2.5" size="0.8128" layer="52" rot="MR90">OE</text>
 </plain>
 <attributes>
@@
 </autorouter>
 <elements>
-<element name="U$1" library="bschulz" package="TSL238T" value="TSL238T" x="7" y="7" smashed="yes"/>
-<element name="H1" library="bschulz" package="2_56" value="" x="2.3" y="12.7" smashed="yes"/>
-<element name="H2" library="bschulz" package="2_56" value="" x="12.7" y="2.3" smashed="yes"/>
-<element name="J1" library="bschulz" package="1X04_NOSILK" value="CONN_42.54_NOSILK" x="6" y="1.2" smashed="yes">
+<element name="U$1" library="bschulz" package="TSL238T" value="TSL238T" x="7" y="7"/>
+<element name="H1" library="bschulz" package="2_56" value="" x="2.3" y="12.7"/>
+<element name="H2" library="bschulz" package="2_56" value="" x="12.7" y="2.3"/>
+<element name="J1" library="bschulz" package="1X04_NOSILK" value="CONN_42.54_NOSILK" x="6" y="1.2">
 <attribute name="NAME" x="4.73" y="2.597" size="0.6096" layer="25" font="vector" ratio="20"/>
 <attribute name="VALUE" x="4.73" y="-0.832" size="0.6096" layer="27" font="vector" ratio="20"/>
 </element>
+<element name="H3" library="bschulz" package="2_56" value="" x="12.7" y="12.7"/>
 </elements>
 <signals>
-<signal name="N$1">
+<signal name="GND">
 <contactref element="U$1" pad="GND"/>
 <contactref element="J1" pad="2"/>
@@
 <wire x1="5.1" y1="1.57" x2="4.73" y2="1.2" width="0.508" layer="1"/>
 </signal>
-<signal name="N$2">
+<signal name="VDD">
 <contactref element="U$1" pad="VDD"/>
 <contactref element="J1" pad="1"/>
@@
 <wire x1="3.6936" y1="8.3683375" x2="3.6936" y2="2.7036" width="0.508" layer="1"/>
 </signal>
-<signal name="N$3">
+<signal name="OE">
 <contactref element="U$1" pad="OE_INV"/>
 <contactref element="J1" pad="3"/>
@@
 <wire x1="7" y1="6.3747375" x2="7" y2="1.47" width="0.508" layer="1"/>
 </signal>
-<signal name="N$4">
+<signal name="OUT">
 <contactref element="U$1" pad="OUT"/>
 <contactref element="J1" pad="4"/>

Commit message: re-center detector
Parts:
- moved U$1 0.71 mm to (7.50, 7.50)
- moved J1 0.64 mm to (5.50, 1.60)
Routing:
- net GND: track 5.20 -> 5.72 mm
- net VDD: track 14.4 -> 14.9 mm
Changed lines of the file:
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@@
 <wire x1="0" y1="13" x2="0" y2="2" width="0" layer="20"/>
 <wire x1="0" y1="2" x2="2" y2="0" width="0" layer="20" curve="90"/>
-<text x="1.8" y="2.5" size="0.8128" layer="52" rot="MR90">VDD</text>
-<text x="9.3" y="2.5" size="0.8128" layer="52" rot="MR90">OUT</text>
-<text x="4.3" y="2.5" size="0.8128" layer="52" rot="MR90">GND</text>
-<text x="6.8" y="2.5" size="0.8128" layer="52" rot="MR90">OE</text>
+<text x="1.3" y="2.9" size="0.8128" layer="52" rot="MR90">VDD</text>
+<text x="8.8" y="2.9" size="0.8128" layer="52" rot="MR90">OUT</text>
+<text x="3.8" y="2.9" size="0.8128" layer="52" rot="MR90">GND</text>
+<text x="6.3" y="2.9" size="0.8128" layer="52" rot="MR90">OE</text>
 </plain>
 <attributes>
@@
 </autorouter>
 <elements>
-<element name="U$1" library="bschulz" package="TSL238T" value="TSL238T" x="7" y="7"/>
+<element name="U$1" library="bschulz" package="TSL238T" value="TSL238T" x="7.5" y="7.5"/>
 <element name="H1" library="bschulz" package="2_56" value="" x="2.3" y="12.7"/>
 <element name="H2" library="bschulz" package="2_56" value="" x="12.7" y="2.3"/>
-<element name="J1" library="bschulz" package="1X04_NOSILK" value="CONN_42.54_NOSILK" x="6" y="1.2">
-<attribute name="NAME" x="4.73" y="2.597" size="0.6096" layer="25" font="vector" ratio="20"/>
-<attribute name="VALUE" x="4.73" y="-0.832" size="0.6096" layer="27" font="vector" ratio="20"/>
+<element name="J1" library="bschulz" package="1X04_NOSILK" value="CONN_42.54_NOSILK" x="5.5" y="1.6">
+<attribute name="NAME" x="4.23" y="2.997" size="0.6096" layer="25" font="vector" ratio="20"/>
+<attribute name="VALUE" x="4.23" y="-0.432" size="0.6096" layer="27" font="vector" ratio="20"/>
 </element>
 <element name="H3" library="bschulz" package="2_56" value="" x="12.7" y="12.7"/>
@@
 <contactref element="U$1" pad="GND"/>
 <contactref element="J1" pad="2"/>
-<wire x1="5.1" y1="6.25" x2="5.1" y2="1.57" width="0.508" layer="1"/>
-<wire x1="5.1" y1="1.57" x2="4.73" y2="1.2" width="0.508" layer="1"/>
+<wire x1="5.6" y1="6.75" x2="5.6" y2="2.97" width="0.4064" layer="1"/>
+<wire x1="5.6" y1="2.97" x2="4.23" y2="1.6" width="0.4064" layer="1"/>
 </signal>
 <signal name="VDD">
 <contactref element="U$1" pad="VDD"/>
 <contactref element="J1" pad="1"/>
-<wire x1="6.5064" y1="8.3683375" x2="6.2683375" y2="8.6064" width="0.508" layer="1"/>
-<wire x1="6.2683375" y1="8.6064" x2="3.9316625" y2="8.6064" width="0.508" layer="1"/>
-<wire x1="3.9316625" y1="8.6064" x2="3.6936" y2="8.3683375" width="0.508" layer="1"/>
-<wire x1="8.9" y1="6.25" x2="8.0586875" y2="6.25" width="0.508" layer="1"/>
-<wire x1="6.5064" y1="7.8022875" x2="6.5064" y2="8.3683375" width="0.508" layer="1"/>
-<wire x1="8.0586875" y1="6.25" x2="6.5064" y2="7.8022875" width="0.508" layer="1"/>
-<wire x1="3.6936" y1="2.7036" x2="2.19" y2="1.2" width="0.508" layer="1"/>
-<wire x1="3.6936" y1="8.3683375" x2="3.6936" y2="2.7036" width="0.508" layer="1"/>
+<wire x1="6.9556" y1="8.84729375" x2="6.74729375" y2="9.0556" width="0.4064" layer="1"/>
+<wire x1="6.74729375" y1="9.0556" x2="4.45270625" y2="9.0556" width="0.4064" layer="1"/>
+<wire x1="4.45270625" y1="9.0556" x2="4.2444" y2="8.84729375" width="0.4064" layer="1"/>
+<wire x1="9.4" y1="6.75" x2="8.3431625" y2="6.75" width="0.4064" layer="1"/>
+<wire x1="6.9556" y1="8.1375625" x2="6.9556" y2="8.84729375" width="0.4064" layer="1"/>
+<wire x1="8.3431625" y1="6.75" x2="6.9556" y2="8.1375625" width="0.4064" layer="1"/>
+<wire x1="4.2444" y1="4.1544" x2="1.69" y2="1.6" width="0.4064" layer="1"/>
+<wire x1="4.2444" y1="8.84729375" x2="4.2444" y2="4.1544" width="0.4064" layer="1"/>
 </signal>
 <signal name="OE">
 <contactref element="U$1" pad="OE_INV"/>
 <contactref element="J1" pad="3"/>
-<wire x1="5.1" y1="7.75" x2="5.7436" y2="7.1064" width="0.508" layer="1"/>
-<wire x1="5.7436" y1="7.1064" x2="6.2683375" y2="7.1064" width="0.508" layer="1"/>
-<wire x1="6.2683375" y1="7.1064" x2="7" y2="6.3747375" width="0.508" layer="1"/>
-<wire x1="7" y1="1.47" x2="7.27" y2="1.2" width="0.508" layer="1"/>
-<wire x1="7" y1="6.3747375" x2="7" y2="1.47" width="0.508" layer="1"/>
+<wire x1="5.6" y1="8.25" x2="6.2944" y2="7.5556" width="0.4064" layer="1"/>
+<wire x1="6.2944" y1="7.5556" x2="6.74729375" y2="7.5556" width="0.4064" layer="1"/>
+<wire x1="6.74729375" y1="7.5556" x2="7" y2="7.30289375" width="0.4064" layer="1"/>
+<wire x1="7" y1="1.83" x2="6.77" y2="1.6" width="0.4064" layer="1"/>
+<wire x1="7" y1="7.30289375" x2="7" y2="1.83" width="0.4064" layer="1"/>
 </signal>
 <signal name="OUT">
 <contactref element="U$1" pad="OUT"/>
 <contactref element="J1" pad="4"/>
-<wire x1="8.9" y1="7.75" x2="9.5436" y2="7.1064" width="0.508" layer="1"/>
-<wire x1="9.5436" y1="7.1064" x2="10.0683375" y2="7.1064" width="0.508" layer="1"/>
-<wire x1="10.0683375" y1="7.1064" x2="10.3064" y2="6.8683375" width="0.508" layer="1"/>
-<wire x1="10.3064" y1="6.8683375" x2="10.3064" y2="5.6316625" width="0.508" layer="1"/>
-<wire x1="9.81" y1="5.1352625" x2="9.81" y2="1.2" width="0.508" layer="1"/>
-<wire x1="10.3064" y1="5.6316625" x2="9.81" y2="5.1352625" width="0.508" layer="1"/>
+<wire x1="9.31" y1="4.31" x2="9.31" y2="1.6" width="0.4064" layer="1"/>
+<wire x1="10.54729375" y1="7.5556" x2="10.7556" y2="7.34729375" width="0.4064" layer="1"/>
+<wire x1="10.0944" y1="7.5556" x2="10.54729375" y2="7.5556" width="0.4064" layer="1"/>
+<wire x1="10.7556" y1="7.34729375" x2="10.7556" y2="5.7556" width="0.4064" layer="1"/>
+<wire x1="9.4" y1="8.25" x2="10.0944" y2="7.5556" width="0.4064" layer="1"/>
+<wire x1="10.7556" y1="5.7556" x2="9.31" y2="4.31" width="0.4064" layer="1"/>
 </signal>
 </signals>
